File: KiCad/PXU.kicad_pcb (KiCad board)
At the start: 4 copper layers, 198 x 64.5 mm, 129 parts, among them IC1 TPS53319DQPT, IC2 TPS53318DQPT, J1 39-38-1203, J2 171826-4, U1 SN74LVC08ADR, U2 LMR33640ADDAR, U3 CSD25402Q3A, U4 AP7375Q-33SP-13, U5 UCC27517A, U6 SN74LVC2G17DBVR

Commit message: License upload
Missed including license in initial upload
Other:
- board text added: "Copyright (C) 2025 Andr0 Licensed under the CERN-OHL-S v2 or later. This documentation is distributed WITHOUT ANY EXPRESS OR IMPLIED WARRANTY, INCLUDING OF MERCHANTABILITY, SATISFACTORY QUALITY AND FITNESS FOR A PARTICULAR PURPOSE. Please see the CERN-OHL-S v2 for details."
Changed lines of the file:
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@@
 		)
 	)
+	(gr_text "Copyright (C) 2025 Andr0\n\nLicensed under the CERN-OHL-S v2 or later.\nThis documentation is distributed WITHOUT ANY EXPRESS OR\nIMPLIED WARRANTY, INCLUDING OF MERCHANTABILITY, SATISFACTORY\nQUALITY AND FITNESS FOR A PARTICULAR PURPOSE. Please see\nthe CERN-OHL-S v2 for details."
+		(at 130.5994 88.8768 0)
+		(layer "User.1")
+		(effects
+			(font
+				(size 1 1)
+				(thickness 0.15)
+			)
+			(justify left bottom)
+		)
+	)
 	(gr_text "{\n  \"ViaStitching\": \"0.2\",\n  \"stitch_zone_0\": {\n    \"HSpacing\": \"5\",\n    \"VSpacing\": \"5\",\n    \"Clearance\": \"0.5\",\n    \"Randomize\": false\n  }\n}"
 		(at 0 0 0)
@@
 			"2789e5ee-7a92-4222-a8c7-21ae8f4675e8" "3dd531dd-f4ea-4a6c-b57f-77289859be35"
 			"4bd94cc8-997a-442a-8b2b-ff978c32e2bd" "5354615a-6af8-4e96-ade6-abf8e0f0844e"
-			"8123f273-3998-4f8b-abc8-42e69aab4dfb" "8f09a6d0-43d3-47c2-b7a9-d3ca0aa47393"
-			"93f631ac-af85-4295-ad35-d0499a433389" "db5cdd14-ac91-4d31-9ca5-6a5fe56b83ee"
+			"8f09a6d0-43d3-47c2-b7a9-d3ca0aa47393" "93f631ac-af85-4295-ad35-d0499a433389"
+			"db5cdd14-ac91-4d31-9ca5-6a5fe56b83ee"
 		)
 	)
